File: design/TechWaveAudio_MidiController.kicad_sch (KiCad schematic)
At the start: 95 parts, among them J1 Control, J10 Midi, J11 PiPico2, J12 PiPico2, J13 Velocity, J14 Note, J2 PowerBus, J3 Aux, J4 Gate, J5 Clock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

Commit message: working multicore
Connections:
- net noteOut: now also SW1.7; no longer SW1.6
- net at SW1.2: now also D2.2 (A)
- net at SW1.3: no longer D2.2 (A)
Other:
- moved on the sheet: D2
Changed lines of the file:
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@@
 	)
 	(no_connect
-		(at 152.4 40.64)
-	)
-	(no_connect
-		(at 167.64 40.64)
-	)
-	(no_connect
 		(at 147.32 80.01)
 	)
@@
 	)
 	(no_connect
+		(at 167.64 43.18)
+	)
+	(no_connect
 		(at 119.38 90.17)
 	)
@@
 	)
 	(no_connect
+		(at 152.4 43.18)
+	)
+	(no_connect
 		(at 224.79 142.24)
 	)
@@
 	(wire
 		(pts
-			(xy 148.59 43.18) (xy 152.4 43.18)
-		)
-		(stroke
-			(width 0)
-			(type default)
-		)
-	)
-	(wire
-		(pts
 			(xy 45.72 30.48) (xy 45.72 33.02)
 		)
@@
 	(wire
 		(pts
+			(xy 148.59 40.64) (xy 152.4 40.64)
+		)
+		(stroke
+			(width 0)
+			(type default)
+		)
+	)
+	(wire
+		(pts
 			(xy 196.85 95.25) (xy 196.85 87.63)
 		)
@@
 	(wire
 		(pts
-			(xy 137.16 43.18) (xy 140.97 43.18)
-		)
-		(stroke
-			(width 0)
-			(type default)
-		)
-	)
-	(wire
-		(pts
 			(xy 147.32 171.45) (xy 147.32 173.99)
 		)
@@
 	(wire
 		(pts
+			(xy 137.16 40.64) (xy 140.97 40.64)
+		)
+		(stroke
+			(width 0)
+			(type default)
+		)
+	)
+	(wire
+		(pts
 			(xy 130.81 147.32) (xy 144.78 147.32)
 		)
@@
 	(global_label "noteOut"
 		(shape input)
-		(at 167.64 43.18 0)
+		(at 167.64 40.64 0)
 		(fields_autoplaced yes)
 		(effects
@@
 		)
 		(property "Intersheetrefs" "${INTERSHEET_REFS}"
-			(at 177.9427 43.18 0)
+			(at 177.9427 40.64 0)
 			(hide yes)
 			(show_name no)
@@
 	(global_label "cvBus"
 		(shape input)
-		(at 137.16 43.18 180)
+		(at 137.16 40.64 180)
 		(fields_autoplaced yes)
 		(effects
@@
 		)
 		(property "Intersheetrefs" "${INTERSHEET_REFS}"
-			(at 128.6715 43.18 0)
+			(at 128.6715 40.64 0)
 			(hide yes)
 			(show_name no)
@@
 	(symbol
 		(lib_id "Device:D_Schottky")
-		(at 144.78 43.18 0)
+		(at 144.78 40.64 0)
 		(unit 1)
 		(body_style 1)
@@
 		(dnp no)
 		(property "Reference" "D2"
-			(at 144.78 46.736 0)
+			(at 144.78 43.434 0)
 			(show_name no)
 			(do_not_autoplace no)
@@
 		)
 		(property "Value" "30V,Schottky"
-			(at 144.78 49.276 0)
+			(at 144.78 45.974 0)
 			(show_name no)
 			(do_not_autoplace no)
@@
 		)
 		(property "Footprint" "Package_TO_SOT_SMD:SOT-23"
-			(at 144.78 43.18 0)
+			(at 144.78 40.64 0)
 			(hide yes)
 			(show_name no)
@@
 		)
 		(property "Datasheet" ""
-			(at 144.78 43.18 0)
+			(at 144.78 40.64 0)
 			(hide yes)
 			(show_name no)
@@
 		)
 		(property "Description" "Schottky diode"
-			(at 144.78 43.18 0)
+			(at 144.78 40.64 0)
 			(hide yes)
 			(show_name no)

Commit message: PCB update; cleanups
Parts:
- added C21, C24: 10uF, Capacitor_SMD:C_0805_2012Metric, symbol Device:C_Polarized
- added C22, C23: 100nf, Capacitor_SMD:C_0402_1005Metric, symbol Device:C
- J9: now fitted
- R37, R39, R41, R43: footprint Resistor_THT:Bourns 3306P-1-102 Trimmer Resistor -> Potentiometer_THT:Potentiometer_Piher_PT-10-V10_Vertical; now fitted
Connections:
- net +12V: now also C21.1, C22.1, C23.1, C24.1
- net GND: now also C21.2, C22.2, C23.2, C24.2
Other:
- moved on the sheet: U1E, U2E

Commit message: doc cleanups and add images
Parts:
- D10, D11, D9: footprint Connector_PinHeader_2.54mm:PinHeader_1x02_P2.54mm_Vertical -> LED_THT:LED_Rectangular_W5.0mm_H2.0mm
- R37, R39, R41, R43: footprint Potentiometer_THT:Potentiometer_Piher_PT-10-V10_Vertical -> Potentiometer_THT:Potentiometer_Bourns_3296X_Horizontal
Changed lines of the file:
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@@
 			)
 		)
-		(property "Footprint" "Potentiometer_THT:Potentiometer_Piher_PT-10-V10_Vertical"
+		(property "Footprint" "Potentiometer_THT:Potentiometer_Bourns_3296X_Horizontal"
 			(at 247.65 46.99 0)
 			(hide yes)
@@
 			)
 		)
-		(property "Footprint" "Connector_PinHeader_2.54mm:PinHeader_1x02_P2.54mm_Vertical"
+		(property "Footprint" "LED_THT:LED_Rectangular_W5.0mm_H2.0mm"
 			(at 245.11 105.41 0)
 			(hide yes)
@@
 			)
 		)
-		(property "Footprint" "Connector_PinHeader_2.54mm:PinHeader_1x02_P2.54mm_Vertical"
+		(property "Footprint" "LED_THT:LED_Rectangular_W5.0mm_H2.0mm"
 			(at 245.11 77.47 0)
 			(hide yes)
@@
 			)
 		)
-		(property "Footprint" "Connector_PinHeader_2.54mm:PinHeader_1x02_P2.54mm_Vertical"
+		(property "Footprint" "LED_THT:LED_Rectangular_W5.0mm_H2.0mm"
 			(at 245.11 110.49 0)
 			(hide yes)
@@
 			)
 		)
-		(property "Footprint" "Potentiometer_THT:Potentiometer_Piher_PT-10-V10_Vertical"
+		(property "Footprint" "Potentiometer_THT:Potentiometer_Bourns_3296X_Horizontal"
 			(at 46.99 127 0)
 			(hide yes)
@@
 			)
 		)
-		(property "Footprint" "Potentiometer_THT:Potentiometer_Piher_PT-10-V10_Vertical"
+		(property "Footprint" "Potentiometer_THT:Potentiometer_Bourns_3296X_Horizontal"
 			(at 247.65 17.78 0)
 			(hide yes)
@@
 			)
 		)
-		(property "Footprint" "Potentiometer_THT:Potentiometer_Piher_PT-10-V10_Vertical"
+		(property "Footprint" "Potentiometer_THT:Potentiometer_Bourns_3296X_Horizontal"
 			(at 58.42 142.24 0)
 			(hide yes)

Commit message: hardware docs; cleanups and comments
Connections:
- net GND: now also U1.12 (+)
- no-connect marks 51 -> 50
Changed lines of the file:
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@@
 	)
 	(no_connect
-		(at 82.55 63.5)
-	)
-	(no_connect
 		(at 119.38 97.79)
 	)
@@
 					(unit 1)
 				)
+			)
+		)
+	)
+	(symbol
+		(lib_name "GND_5")
+		(lib_id "power:GND")
+		(at 82.55 63.5 90)
+		(unit 1)
+		(body_style 1)
+		(exclude_from_sim no)
+		(in_bom yes)
+		(on_board yes)
+		(in_pos_files yes)
+		(dnp no)
+		(fields_autoplaced yes)
+		(property "Reference" "#PWR086"
+			(at 88.9 63.5 0)
+			(hide yes)
+			(show_name no)
+			(do_not_autoplace no)
+			(effects
+				(font
+					(size 1.27 1.27)
+				)
+			)
+		)
+		(property "Value" "GND"
+			(at 86.36 63.4999 90)
+			(show_name no)
+			(do_not_autoplace no)
+			(effects
+				(font
+					(size 1.27 1.27)
+				)
+				(justify right)
+			)
+		)
+		(property "Footprint" ""
+			(at 82.55 63.5 0)
+			(hide yes)
+			(show_name no)
+			(do_not_autoplace no)
+			(effects
+				(font
+					(size 1.27 1.27)
+				)
+			)
+		)
+		(property "Datasheet" ""
+			(at 82.55 63.5 0)
+			(hide yes)
+			(show_name no)
+			(do_not_autoplace no)
+			(effects
+				(font
+					(size 1.27 1.27)
+				)
+			)
+		)
+		(property "Description" "Power symbol creates a global label with name \"GND\" , ground"
+			(at 82.55 63.5 0)
+			(hide yes)
+			(show_name no)
+			(do_not_autoplace no)
+			(effects
+				(font
+					(size 1.27 1.27)
+				)
+			)
+		)
+		(pin "1"
+		)
+		(instances
+			(project "TechWaveAudio_MidiController"
+				(path "/573b317e-655b-4032-b57c-d77b689bdb51"
+					(reference "#PWR086")
+					(unit 1)
+				)

Commit message: parts list; update board
Parts:
- U3: value 74HC7016 -> 40106
Other:
- company: (none) -> TechWave Audio
- title: (none) -> TechWave Audio - MCM
Changed lines of the file:
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@@
 	(paper "A4")
 	(title_block
-		(comment 1 "Version 0.1.0")
+		(title "TechWave Audio - MCM")
+		(date "2026-06-30")
+		(rev "rev 1.1.0")
+		(company "TechWave Audio")
+		(comment 1 "Midi Controller Module")
+		(comment 2 "Version 1.1.0")
 	)
 	(junction
@@
 			)
 		)
-		(property "Value" "74HC7016"
+		(property "Value" "40106"
 			(at 109.982 185.674 0)
 			(show_name no)
@@
 			)
 		)
-		(property "Value" "74HC7016"
+		(property "Value" "40106"
 			(at 60.96 167.386 90)
 			(show_name no)
@@
 			)
 		)
-		(property "Value" "74HC7016"
+		(property "Value" "40106"
 			(at 164.338 175.768 0)
 			(show_name no)
@@
 			)
 		)
-		(property "Value" "74HC7016"
+		(property "Value" "40106"
 			(at 128.524 187.96 0)
 			(show_name no)
@@
 			)
 		)
-		(property "Value" "74HC7016"
+		(property "Value" "40106"
 			(at 151.892 183.642 0)
 			(show_name no)
@@
 			)
 		)
-		(property "Value" "74HC7016"
+		(property "Value" "40106"
 			(at 122.428 177.292 0)
 			(show_name no)
@@
 			)
 		)
-		(property "Value" "74HC7016"
+		(property "Value" "40106"
 			(at 70.358 191.516 0)
 			(show_name no)
