File: design/TechWaveAudio_MidiController.kicad_sch (KiCad schematic)
At the start: 99 parts, among them J1 Control, J10 Midi, J11 PiPico2, J12 PiPico2, J13 Velocity, J14 Note, J2 PowerBus, J3 Aux, J4 Gate, J5 Clock, J6 Trigger, J7 PiPico1, J8 PiPico1, J9 5WaySwitch, SW1 SW_DIP_x04, U1 TL074, U2 TL074, U3 40106, U4 MCP4902, U5 MCP4725, U6 MCP4725, U7 6N137

Commit message: latest board design
Parts:
- J1, J13, J14, J3, J4, J5, J6: footprint Connector_PinHeader_2.54mm:PinHeader_1x02_P2.54mm_Vertical -> Connector_Audio:Jack_3.5mm_SameSky_SJ3-3505x
Changed lines of the file:
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@@
 			)
 		)
-		(property "Footprint" "Connector_PinHeader_2.54mm:PinHeader_1x02_P2.54mm_Vertical"
+		(property "Footprint" "Connector_Audio:Jack_3.5mm_SameSky_SJ3-3505x"
 			(at 33.02 118.11 0)
 			(hide yes)
@@
 			)
 		)
-		(property "Footprint" "Connector_PinHeader_2.54mm:PinHeader_1x02_P2.54mm_Vertical"
+		(property "Footprint" "Connector_Audio:Jack_3.5mm_SameSky_SJ3-3505x"
 			(at 259.08 26.67 0)
 			(hide yes)
@@
 			)
 		)
-		(property "Footprint" "Connector_PinHeader_2.54mm:PinHeader_1x02_P2.54mm_Vertical"
+		(property "Footprint" "Connector_Audio:Jack_3.5mm_SameSky_SJ3-3505x"
 			(at 57.15 92.71 0)
 			(hide yes)
@@
 			)
 		)
-		(property "Footprint" "Connector_PinHeader_2.54mm:PinHeader_1x02_P2.54mm_Vertical"
+		(property "Footprint" "Connector_Audio:Jack_3.5mm_SameSky_SJ3-3505x"
 			(at 57.15 80.01 0)
 			(hide yes)
@@
 			)
 		)
-		(property "Footprint" "Connector_PinHeader_2.54mm:PinHeader_1x02_P2.54mm_Vertical"
+		(property "Footprint" "Connector_Audio:Jack_3.5mm_SameSky_SJ3-3505x"
 			(at 44.45 133.35 0)
 			(hide yes)
@@
 			)
 		)
-		(property "Footprint" "Connector_PinHeader_2.54mm:PinHeader_1x02_P2.54mm_Vertical"
+		(property "Footprint" "Connector_Audio:Jack_3.5mm_SameSky_SJ3-3505x"
 			(at 256.54 55.88 0)
 			(hide yes)
@@
 			)
 		)
-		(property "Footprint" "Connector_PinHeader_2.54mm:PinHeader_1x02_P2.54mm_Vertical"
+		(property "Footprint" "Connector_Audio:Jack_3.5mm_SameSky_SJ3-3505x"
 			(at 57.15 105.41 0)
 			(hide yes)
