File: design/TechWaveAudio_MidiController.kicad_pcb (KiCad board)
At the start: 2 copper layers, 111.5 x 128.5 mm, 96 parts, among them J1 Control, J10 Midi, J12 PiPico2, J13 Velocity, J14 Note, J2 PowerBus, J3 Aux, J4 Gate, J5 Clock, J6 Trigger, J7 PiPico1, J9 5WaySwitch, SW1 SW_DIP_x04, U1 TL074, U2 TL074, U3 74HC7016, U4 MCP4902, U5 MCP4725, U6 MCP4725, U7 6N137

Commit message: latest board design
Parts:
- J1, J13, J14, J3, J4, J5, J6: footprint Connector_PinHeader_2.54mm:PinHeader_1x02_P2.54mm_Vertical -> Connector_Audio:Jack_3.5mm_SameSky_SJ3-3505x
- U3: value 74HC7016 -> 40106
- moved R37 33.5 mm to (122.0, 38.7)
- moved R30 23.3 mm to (129.4, 47.0), turned to 90 degrees
- moved R7 23.0 mm to (122.4, 46.5), turned to 0 degrees
- moved R10 22.0 mm to (114.7, 114.0), turned to 180 degrees
- moved R6 21.9 mm to (116.5, 115.0)
- moved J5 21.4 mm to (137.3, 115.2), turned to 0 degrees
- moved R27 20.8 mm to (128.2, 47.0), turned to -90 degrees
- moved R40 19.5 mm to (122.4, 49.4), turned to 90 degrees
- moved R5 19.3 mm to (125.5, 107.2)
- moved U2 17.3 mm to (126.9, 52.9), turned to 0 degrees
- moved R9 17.0 mm to (125.0, 105.5)
- moved R28 16.8 mm to (129.4, 58.8), turned to 90 degrees
- moved C8 16.5 mm to (125.2, 39.7), turned to 90 degrees
- moved U1 15.8 mm to (120.2, 110.2), turned to -90 degrees
- moved R38 14.6 mm to (128.2, 58.8), turned to -90 degrees
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Routing:
- net +5V: track 217.4 -> 261.9 mm, vias 4 -> 3
- net /ctlDACOut: track 62.0 -> 32.8 mm
- net /auxDACOut: track 61.5 -> 32.3 mm
- net -12V: track 102.8 -> 125.9 mm
- net +12V: track 96.6 -> 116.1 mm, vias 4 -> 2
- net /auxOut: track 45.6 -> 26.3 mm, vias 2 -> 1
- net /trg: track 22.9 -> 39.4 mm, vias 0 -> 1
- net Net-(R30-Pad2): track 29.9 -> 14.0 mm, vias 1 -> 2
- net /gate: track 33.0 -> 47.9 mm
- net Net-(R38-Pad2): track 18.5 -> 29.3 mm, vias 1 -> 0
- net noteOut: track 122.8 -> 112.0 mm, vias 2 -> 1
- net /4725Clk: track 24.1 -> 34.0 mm
- net cvBus: track 14.5 -> 24.2 mm
- net gateOut: track 54.9 -> 63.8 mm, vias 2 -> 3
- net /4902Clk: track 13.6 -> 5.07 mm
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Other:
- board size 111.5 x 128.5 mm -> 120.8 x 128.5 mm
- board text added: "MCM-100"
- board text added: "audio"
- board text added: "techwave"
