File: design/TechWaveAudio-MCM-100-PCB/TechWaveAudio_MidiController.kicad_sch (KiCad schematic)
At the start: 99 parts, among them J1 Control, J10 Midi, J11 PiPico2, J12 PiPico2, J13 Velocity, J14 Note, J2 PowerBus, J3 Aux, J4 Gate, J5 Clock, J6 Trigger, J7 PiPico1, J8 PiPico1, J9 5WaySwitch, SW1 SW_DIP_x04, U1 TL074, U2 TL074, U3 40106, U4 MCP4902, U5 MCP4725, U6 MCP4725, U7 6N137

Commit message: move PCB and panel to separate folders
Other:
- title: TechWave Audio - MCM -> TechWave Audio - MCM-100
- moved on the sheet: C21, C22, U1E
Changed lines of the file:
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@@
 	(paper "A4")
 	(title_block
-		(title "TechWave Audio - MCM")
-		(date "2026-06-30")
-		(rev "rev 1.1.0")
+		(title "TechWave Audio - MCM-100")
+		(date "2026-07-14")
+		(rev "v 1.2.0")
 		(company "TechWave Audio")
 		(comment 1 "Midi Controller Module")
-		(comment 2 "Version 1.1.0")
+		(comment 2 "Version 1.2.0")
 	)
 	(junction
@@
 	)
 	(junction
+		(at 25.4 81.28)
+		(diameter 0)
+		(color 0 0 0 0)
+	)
+	(junction
 		(at 33.02 27.94)
 		(diameter 0)
@@
 	)
 	(junction
-		(at 26.035 86.36)
-		(diameter 0)
-		(color 0 0 0 0)
-	)
-	(junction
 		(at 256.54 107.95)
 		(diameter 0)
@@
 	)
 	(junction
+		(at 25.4 86.36)
+		(diameter 0)
+		(color 0 0 0 0)
+	)
+	(junction
 		(at 187.96 29.21)
 		(diameter 0)
@@
 	)
 	(junction
-		(at 26.035 81.28)
-		(diameter 0)
-		(color 0 0 0 0)
-	)
-	(junction
 		(at 62.23 77.47)
 		(diameter 0)
@@
 	(wire
 		(pts
-			(xy 26.035 81.28) (xy 23.495 81.28)
+			(xy 72.39 118.11) (xy 72.39 125.73)
 		)
 		(stroke
@@
 	(wire
 		(pts
-			(xy 72.39 118.11) (xy 72.39 125.73)
+			(xy 144.78 147.32) (xy 144.78 156.21)
 		)
 		(stroke
@@
 	(wire
 		(pts
-			(xy 144.78 147.32) (xy 144.78 156.21)
+			(xy 26.67 50.8) (xy 38.1 50.8)
 		)
 		(stroke
@@
 	(wire
 		(pts
-			(xy 26.67 50.8) (xy 38.1 50.8)
+			(xy 190.5 17.78) (xy 189.23 17.78)
 		)
 		(stroke
@@
 	(wire
 		(pts
-			(xy 190.5 17.78) (xy 189.23 17.78)
+			(xy 210.82 69.85) (xy 214.63 69.85)
 		)
 		(stroke
@@
 	(wire
 		(pts
-			(xy 210.82 69.85) (xy 214.63 69.85)
+			(xy 25.4 81.28) (xy 25.4 86.36)
 		)
 		(stroke
@@
 	(wire
 		(pts
-			(xy 26.035 86.36) (xy 26.035 81.28)
-		)
-		(stroke
-			(width 0)
-			(type default)
-		)
-	)
-	(wire
-		(pts
 			(xy 220.98 144.78) (xy 224.79 144.78)
 		)
@@
 	(wire
 		(pts
-			(xy 28.575 81.28) (xy 26.035 81.28)
-		)
-		(stroke
-			(width 0)
-			(type default)
-		)
-	)
-	(wire
-		(pts
 			(xy 100.33 52.07) (xy 100.33 53.34)
 		)
@@
 	(wire
 		(pts
+			(xy 25.4 81.28) (xy 29.21 81.28)
+		)
+		(stroke
+			(width 0)
+			(type default)
+		)
+	)
+	(wire
+		(pts
 			(xy 119.38 113.03) (xy 110.49 113.03)
 		)
@@
 	(wire
 		(pts
+			(xy 24.13 81.28) (xy 25.4 81.28)
+		)
+		(stroke
+			(width 0)
+			(type default)
+		)
+	)
+	(wire
+		(pts
 			(xy 137.16 40.64) (xy 140.97 40.64)
 		)
@@
 	(symbol
 		(lib_id "power:GND")
-		(at 23.495 73.66 180)
+		(at 24.13 73.66 180)
 		(unit 1)
 		(body_style 1)
@@
 		(dnp no)
 		(property "Reference" "#PWR082"
-			(at 23.495 67.31 0)
+			(at 24.13 67.31 0)
 			(hide yes)
 			(show_name no)
@@
 		)
 		(property "Value" "GND"
-			(at 26.035 73.025 90)
+			(at 26.67 73.025 90)
 			(show_name no)
 			(do_not_autoplace no)
@@
 		)
 		(property "Footprint" ""
-			(at 23.495 73.66 0)
+			(at 24.13 73.66 0)
 			(hide yes)
 			(show_name no)
@@
 		)
 		(property "Datasheet" ""
-			(at 23.495 73.66 0)
+			(at 24.13 73.66 0)
 			(hide yes)
 			(show_name no)
@@
 		)
 		(property "Description" ""
-			(at 23.495 73.66 0)
+			(at 24.13 73.66 0)
 			(show_name no)
 			(do_not_autoplace no)
@@
 	(symbol
 		(lib_id "Amplifier_Operational:TL074")
-		(at 33.655 83.82 90)
+		(at 33.02 83.82 90)
 		(unit 5)
 		(body_style 1)
@@
 		(fields_autoplaced yes)
 		(property "Reference" "U1"
-			(at 33.655 81.28 90)
+			(at 33.02 81.28 90)
 			(show_name no)
 			(do_not_autoplace no)
@@
 		)
 		(property "Value" "TL074"
-			(at 33.655 83.82 90)
+			(at 33.02 83.82 90)
 			(show_name no)
 			(do_not_autoplace no)
@@
 		)
 		(property "Footprint" "Package_SO:SOIC-14_3.9x8.7mm_P1.27mm"
-			(at 31.115 85.09 0)
+			(at 30.48 85.09 0)
 			(hide yes)
 			(show_name no)
@@
 		)
 		(property "Datasheet" "http://www.ti.com/lit/ds/symlink/tl071.pdf"
-			(at 28.575 82.55 0)
+			(at 27.94 82.55 0)
 			(hide yes)
 			(show_name no)
@@
 		)
 		(property "Description" "Quad Low-Noise JFET-Input Operational Amplifiers, DIP-14/SOIC-14"
-			(at 33.655 83.82 0)
+			(at 33.02 83.82 0)
 			(hide yes)
 			(show_name no)
@@
 		)
 		(property "BriefDescription" ""
-			(at 33.655 83.82 90)
+			(at 33.02 83.82 90)
 			(hide yes)
 			(show_name no)
@@
 	(symbol
 		(lib_id "power:+12V")
-		(at 26.035 86.36 90)
+		(at 25.4 86.36 90)
 		(unit 1)
 		(body_style 1)
@@
 		(fields_autoplaced yes)
 		(property "Reference" "#PWR03"
-			(at 29.845 86.36 0)
+			(at 29.21 86.36 0)
 			(hide yes)
 			(show_name no)
@@
 		)
 		(property "Value" "+12V"
-			(at 22.225 86.3599 90)
+			(at 21.59 86.3599 90)
 			(show_name no)
 			(do_not_autoplace no)
@@
 		)
 		(property "Footprint" ""
-			(at 26.035 86.36 0)
+			(at 25.4 86.36 0)
 			(hide yes)
 			(show_name no)
@@
 		)
 		(property "Datasheet" ""
-			(at 26.035 86.36 0)
+			(at 25.4 86.36 0)
 			(hide yes)
 			(show_name no)
@@
 		)
 		(property "Description" "Power symbol creates a global label with name \"+12V\""
-			(at 26.035 86.36 0)
+			(at 25.4 86.36 0)
 			(hide yes)
 			(show_name no)
@@
 	(symbol
 		(lib_id "Device:C_Polarized")
-		(at 28.575 77.47 180)
+		(at 29.21 77.47 180)
 		(unit 1)
 		(body_style 1)
@@
 		(dnp no)
 		(property "Reference" "C21"
-			(at 35.941 78.486 0)
+			(at 36.576 78.486 0)
 			(show_name no)
 			(do_not_autoplace no)
@@
 		)
 		(property "Value" "10uF"
-			(at 35.941 75.946 0)
+			(at 36.576 75.946 0)
 			(show_name no)
 			(do_not_autoplace no)
@@
 		)
 		(property "Footprint" "Capacitor_SMD:C_0805_2012Metric"
-			(at 27.6098 73.66 0)
+			(at 28.2448 73.66 0)
 			(hide yes)
 			(show_name no)
@@
 		)
 		(property "Datasheet" ""
-			(at 28.575 77.47 0)
+			(at 29.21 77.47 0)
 			(hide yes)
 			(show_name no)
@@
 		)
 		(property "Description" "Polarized capacitor"
-			(at 28.575 77.47 0)
+			(at 29.21 77.47 0)
 			(hide yes)
 			(show_name no)
@@
 	(symbol
 		(lib_id "power:-12V")
-		(at 41.275 86.36 270)
+		(at 40.64 86.36 270)
 		(unit 1)
 		(body_style 1)
@@
 		(fields_autoplaced yes)
 		(property "Reference" "#PWR02"
-			(at 37.465 86.36 0)
+			(at 36.83 86.36 0)
 			(hide yes)
 			(show_name no)
@@
 		)
 		(property "Value" "-12V"
-			(at 45.085 86.3599 90)
+			(at 44.45 86.3599 90)
 			(show_name no)
 			(do_not_autoplace no)
@@
 		)
 		(property "Footprint" ""
-			(at 41.275 86.36 0)
+			(at 40.64 86.36 0)
 			(hide yes)
 			(show_name no)
@@
 		)
 		(property "Datasheet" ""
-			(at 41.275 86.36 0)
+			(at 40.64 86.36 0)
 			(hide yes)
 			(show_name no)
@@
 		)
 		(property "Description" "Power symbol creates a global label with name \"-12V\""
-			(at 41.275 86.36 0)
+			(at 40.64 86.36 0)
 			(hide yes)
 			(show_name no)
@@
 	(symbol
 		(lib_id "Device:C")
-		(at 23.495 77.47 180)
+		(at 24.13 77.47 180)
 		(unit 1)
 		(body_style 1)
@@
 		(fields_autoplaced yes)
 		(property "Reference" "C22"
-			(at 19.685 78.7401 0)
+			(at 20.32 78.7401 0)
 			(show_name no)
 			(do_not_autoplace no)
@@
 		)
 		(property "Value" "100nf"
-			(at 19.685 76.2001 0)
+			(at 20.32 76.2001 0)
 			(show_name no)
 			(do_not_autoplace no)
@@
 		)
 		(property "Footprint" "Capacitor_SMD:C_0402_1005Metric"
-			(at 22.5298 73.66 0)
+			(at 23.1648 73.66 0)
 			(hide yes)
 			(show_name no)
@@
 		)
 		(property "Datasheet" ""
-			(at 23.495 77.47 0)
+			(at 24.13 77.47 0)
 			(hide yes)
 			(show_name no)
@@
 		)
 		(property "Description" "Unpolarized capacitor"
-			(at 23.495 77.47 0)
+			(at 24.13 77.47 0)
 			(hide yes)
 			(show_name no)
@@
 	(symbol
 		(lib_id "power:GND")
-		(at 28.575 73.66 180)
+		(at 29.21 73.66 180)
 		(unit 1)
 		(body_style 1)
@@
 		(dnp no)
 		(property "Reference" "#PWR083"
-			(at 28.575 67.31 0)
+			(at 29.21 67.31 0)
 			(hide yes)
 			(show_name no)
@@
 		)
 		(property "Value" "GND"
-			(at 31.115 73.025 90)
+			(at 31.75 73.025 90)
 			(show_name no)
 			(do_not_autoplace no)
@@
 		)
 		(property "Footprint" ""
-			(at 28.575 73.66 0)
+			(at 29.21 73.66 0)
 			(hide yes)
 			(show_name no)
@@
 		)
 		(property "Datasheet" ""
-			(at 28.575 73.66 0)
+			(at 29.21 73.66 0)
 			(hide yes)
 			(show_name no)
@@
 		)
 		(property "Description" ""
-			(at 28.575 73.66 0)
+			(at 29.21 73.66 0)
 			(show_name no)
 			(do_not_autoplace no)
