File: design/TechWaveAudio-MCM-100-Expansion/TechWaveAudio-MCM-100-EX.kicad_sch (KiCad schematic)
At the start: 19 parts, among them J21 Expansion, J22 xCV1, J23 xCV2, J24 xCV3, J25 xCV4, U1 DAC7554, U2 TL072, U3 TL072

Commit message: update expansion;  ensure ex state is properly set
Parts:
- added D1: LED, LED_THT:LED_D3.0mm, symbol Device:LED
- added R26: 1k, Resistor_SMD:R_0402_1005Metric, symbol Device:R_US
Connections:
- net +5V: now also D1.2 (A)
- net GND: now also J23.1 (Pin_1), R26.2; no longer J23.2 (Pin_2)
- net at R43.1, U3.7: now also J23.2 (Pin_2); no longer J23.1 (Pin_1)
- new net: D1.1 (K), R26.1
Other:
- moved on the sheet: R25
