File: design/TechWaveAudio-MCM-100-PCB-IO/TechWaveAudio_MidiController.kicad_pcb (KiCad board)
At the start: 2 copper layers, 30 x 90 mm, 41 parts, among them J13 Velocity, J14 Note, J15 IO_OLED/DacOut, J19 IO_GateClkTrg, J2 Aux, J3 Control, J4 Gate, J5 Clock, J6 Trigger, J9 IO_EncClkNoteConn, SW1 RotaryEncoder_Switch, U1 TL074, U2 TL074

Commit message: better 7554 ; spi; i2c control; test all outputs selection
Connections:
- D11 pad 1: NoteLed -> Net-(D11-K)
- D11 pad 2: Net-(D11-A) -> NoteLed
- R38 pad 1: Net-(D11-A) -> Net-(D11-K)
Routing:
- net NoteLed: track 12.8 -> 9.35 mm
- net Net-(D11-A): track 2.73 -> 0.00 mm
- net Net-(D11-K): track 0.00 -> 2.39 mm
Changed lines of the file:
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@@
 			)
 		)
-		(attr through_hole exclude_from_pos_files exclude_from_bom)
+		(attr through_hole)
 		(duplicate_pad_numbers_are_jumpers no)
 		(fp_line
@@
 			)
 		)
-		(attr through_hole exclude_from_pos_files exclude_from_bom)
+		(attr through_hole)
 		(duplicate_pad_numbers_are_jumpers no)
 		(fp_line
@@
 			)
 		)
-		(attr through_hole exclude_from_pos_files exclude_from_bom)
+		(attr through_hole)
 		(duplicate_pad_numbers_are_jumpers no)
 		(fp_line
@@
 			)
 		)
-		(attr smd exclude_from_pos_files exclude_from_bom)
+		(attr smd)
 		(duplicate_pad_numbers_are_jumpers no)
 		(fp_rect
@@
 			(layers "F.Cu" "F.Mask" "F.Paste")
 			(roundrect_rratio 0.25)
-			(net "Net-(D11-A)")
+			(net "Net-(D11-K)")
 			(pintype "passive")
 		)
@@
 			)
 		)
-		(attr exclude_from_pos_files exclude_from_bom)
+		(attr exclude_from_bom)
 		(duplicate_pad_numbers_are_jumpers no)
 		(fp_circle
@@
 			)
 		)
-		(attr through_hole exclude_from_pos_files exclude_from_bom)
+		(attr through_hole exclude_from_bom)
 		(duplicate_pad_numbers_are_jumpers no)
 		(fp_line
@@
 			)
 		)
-		(attr through_hole exclude_from_pos_files exclude_from_bom)
+		(attr through_hole exclude_from_bom)
 		(duplicate_pad_numbers_are_jumpers no)
 		(fp_line
@@
 			)
 		)
-		(attr through_hole exclude_from_pos_files exclude_from_bom)
+		(attr through_hole exclude_from_bom)
 		(duplicate_pad_numbers_are_jumpers no)
 		(fp_line
@@
 			)
 		)
-		(attr through_hole exclude_from_pos_files exclude_from_bom)
+		(attr through_hole exclude_from_bom)
 		(duplicate_pad_numbers_are_jumpers no)
 		(fp_line
@@
 			)
 		)
-		(attr through_hole exclude_from_pos_files exclude_from_bom)
+		(attr through_hole exclude_from_bom)
 		(duplicate_pad_numbers_are_jumpers no)
 		(fp_line
@@
 			)
 		)
-		(attr through_hole exclude_from_pos_files exclude_from_bom)
+		(attr through_hole exclude_from_bom)
 		(duplicate_pad_numbers_are_jumpers no)
 		(fp_line
@@
 			)
 		)
-		(attr through_hole exclude_from_pos_files exclude_from_bom)
+		(attr through_hole exclude_from_bom)
 		(duplicate_pad_numbers_are_jumpers no)
 		(fp_line
@@
 			)
 		)
-		(attr through_hole exclude_from_pos_files exclude_from_bom)
+		(attr through_hole exclude_from_bom)
 		(duplicate_pad_numbers_are_jumpers no)
 		(fp_line
@@
 			)
 		)
-		(attr through_hole exclude_from_pos_files exclude_from_bom)
+		(attr through_hole exclude_from_bom)
 		(duplicate_pad_numbers_are_jumpers no)
 		(fp_line
@@
 			)
 		)
-		(attr through_hole exclude_from_pos_files exclude_from_bom)
+		(attr through_hole exclude_from_bom)
 		(duplicate_pad_numbers_are_jumpers no)
 		(fp_line
@@
 			)
 		)
-		(attr through_hole exclude_from_pos_files exclude_from_bom)
+		(attr through_hole exclude_from_bom)
 		(duplicate_pad_numbers_are_jumpers no)
 		(fp_line
@@
 			)
 		)
-		(attr through_hole exclude_from_pos_files exclude_from_bom)
+		(attr through_hole exclude_from_bom)
 		(duplicate_pad_numbers_are_jumpers no)
 		(fp_line
@@
 			)
 		)
-		(attr through_hole exclude_from_pos_files exclude_from_bom)
+		(attr through_hole exclude_from_bom)
 		(duplicate_pad_numbers_are_jumpers no)
 		(fp_line
@@
 			(layers "*.Cu" "*.Mask")
 			(remove_unused_layers no)
-			(net "NoteLed")
+			(net "Net-(D11-K)")
 			(pinfunction "K_1")
 			(pintype "passive")
@@
 			(layers "*.Cu" "*.Mask")
 			(remove_unused_layers no)
-			(net "Net-(D11-A)")
+			(net "NoteLed")
 			(pinfunction "A_2")
 			(pintype "passive")
@@
 			)
 		)
-		(attr through_hole exclude_from_pos_files exclude_from_bom)
+		(attr through_hole exclude_from_bom)
 		(duplicate_pad_numbers_are_jumpers no)
 		(fp_line
@@
 			)
 		)
-		(attr through_hole exclude_from_pos_files exclude_from_bom)
+		(attr through_hole exclude_from_bom)
 		(duplicate_pad_numbers_are_jumpers no)
 		(fp_line
@@
 	)
 	(segment
-		(start 22.47 72.02)
-		(end 23.695 70.795)
-		(width 0.25)
-		(layer "F.Cu")
-		(net "NoteLed")
-	)
-	(segment
-		(start 29.661499 70.795)
-		(end 30.814499 71.948)
-		(width 0.25)
-		(layer "F.Cu")
-		(net "NoteLed")
-	)
-	(segment
 		(start 33.8412 70.773)
-		(end 32.6662 71.948)
-		(width 0.25)
-		(layer "F.Cu")
-		(net "NoteLed")
-	)
-	(segment
-		(start 23.695 70.795)
-		(end 29.661499 70.795)
+		(end 32.5942 72.02)
 		(width 0.25)
 		(layer "F.Cu")
@@
 	)
 	(segment
-		(start 30.814499 71.948)
-		(end 32.6662 71.948)
+		(start 32.5942 72.02)
+		(end 25.01 72.02)
 		(width 0.25)
 		(layer "F.Cu")
@@
 	)
 	(segment
-		(start 23.3304 73.6996)
-		(end 23.3304 74.052)
-		(width 0.25)
-		(layer "F.Cu")
-		(net "Net-(D11-A)")
-	)
-	(segment
-		(start 25.01 72.02)
-		(end 23.3304 73.6996)
-		(width 0.25)
-		(layer "F.Cu")
-		(net "Net-(D11-A)")
-	)
-	(segment
 		(start 32.4584 104.7328)
 		(end 32.4584 106.0028)
@@
 		(net "/Aux2Out")
 	)
+	(segment
+		(start 22.47 72.02)
+		(end 22.47 73.1916)
+		(width 0.25)
+		(layer "F.Cu")
+		(net "Net-(D11-K)")
+	)
+	(segment
+		(start 22.47 73.1916)
+		(end 23.3304 74.052)
+		(width 0.25)
+		(layer "F.Cu")
+		(net "Net-(D11-K)")
+	)
 	(zone
