File: design/TechWaveAudio-MCM-100-PCB-IO/TechWaveAudio_MidiController.kicad_sch (KiCad schematic)
At the start: 41 parts, among them J13 Velocity, J14 Note, J15 IO_OLED/DacOut, J19 IO_GateClkTrg, J2 Aux, J3 Control, J4 Gate, J5 Clock, J6 Trigger, J9 IO_EncClkNoteConn, SW1 RotaryEncoder_Switch, U1 TL074, U2 TL074

Commit message: better 7554 ; spi; i2c control; test all outputs selection
Connections:
- net NoteLed: now also D11.2 (A); no longer D11.1 (K)
- net at R38.1: now also D11.1 (K); no longer D11.2 (A)
Other:
- moved on the sheet: D11
Changed lines of the file:
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@@
 		(lib_id "Device:LED")
 		(at 101.6 48.26 0)
+		(mirror y)
 		(unit 1)
 		(body_style 1)
@@
 		(dnp no)
 		(property "Reference" "D11"
-			(at 100.33 53.34 0)
+			(at 101.6 54.102 0)
 			(show_name no)
 			(do_not_autoplace no)
@@
 		)
 		(property "Value" "Note On"
-			(at 100.33 51.562 0)
+			(at 102.616 51.816 0)
 			(show_name no)
 			(do_not_autoplace no)
